File: Project Blaide/Prototype_001/Electronic/Prototype_001/Prototype_001.kicad_pcb (KiCad board)
At the start: 2 copper layers, 197 parts

Commit message: Ivan - Update: v0.0.0.1 - Finalizing electronic Board
Parts:
- added J1: Connector, Connector_PinHeader_2.54mm:PinHeader_1x06_P2.54mm_Vertical, F.Cu at (76.2, 100.1)
- added J2: Connector, Connector_PinHeader_2.54mm:PinHeader_1x15_P2.54mm_Vertical, F.Cu at (219.8, 44.5)
Routing:
- net row_0: track 0.00 -> 424.8 mm
- net col_0: track 0.00 -> 112.1 mm
- net Net-(D1-A): track 0.00 -> 4.28 mm
